File: RL78_F14_32p_Rev2/RL78_F14_32p_Rev2.kicad_sch (KiCad schematic)
At the start: 39 parts, among them P1 POWER_JACKPTH, P2 E2 Lite, P3 F09HP, P4 Keypad, P5 LCD-1.8, P6 SD_Connector, P8 SPI_to_eth, U1 R5F10PBELNA, U2 AMS1117-3.3, U4 MCP2562FD

Commit message: Fixed errors for Keypad for RL78 F14 board with on board CAN Ports 12.1 and 12.2 do no provide pullups but Port 6.0 and 6.1 do Resistors removed for port 6 since internal pullups can be used Basically the wrong project was copied on github
Parts:
- removed R7, R8: 10k, Resistor_SMD:R_0805_2012Metric, symbol Device:R_US
- renumbered R9 to R7
Connections:
- net +3.3V: now also R5.1, R6.1
- net Key3: now reaches U1.11 (P60)
- net Key3: now also P4.3 (Pin_3)
- net Key4: now reaches U1.12 (P61)
- net Key4: now also P4.4 (Pin_4)
- net Key1: now reaches U1.6 (P122/X2/EXCLK)
- net Key1: now also P4.1 (Pin_1), R5.2; no longer R5.1
- net Key2: now reaches U1.7 (P121/X1)
- net Key2: now also P4.2 (Pin_2), R6.2; no longer R6.1
Other:
- moved on the sheet: P4, R5, R6
