File: RL78_F14_32p_Rev2/RL78_F14_32p_Rev2.kicad_pcb (KiCad board)
At the start: 2 copper layers, 100 x 100 mm, 39 parts, among them P1 POWER_JACKPTH, P2 E2 Lite, P3 F09HP, P4 Keypad, P5 LCD-1.8, P6 SD_Connector, P8 SPI_to_eth, U1 R5F10PBELNA, U2 AMS1117-3.3, U4 MCP2562FD

Commit message: Fixed errors for Keypad for RL78 F14 board with on board CAN Ports 12.1 and 12.2 do no provide pullups but Port 6.0 and 6.1 do Resistors removed for port 6 since internal pullups can be used Basically the wrong project was copied on github
Parts:
- removed the R7 at (109.0, 89.1)
- removed R8: 10k, Resistor_SMD:R_0805_2012Metric
- turned R5 to 180 degrees
- turned R6 to 180 degrees
- renumbered R9 to R7
Connections:
- P4 pad 1: Net-(P4-Pin_1) -> /Key1
- P4 pad 2: Net-(P4-Pin_2) -> /Key2
- P4 pad 3: Net-(P4-Pin_3) -> /Key3
- P4 pad 4: Net-(P4-Pin_4) -> /Key4
- R5 pad 1: Net-(U1-P122/X2/EXCLK) -> +3.3V
- R5 pad 2: Net-(P4-Pin_1) -> /Key1
- R6 pad 1: Net-(U1-P121/X1) -> +3.3V
- R6 pad 2: Net-(P4-Pin_2) -> /Key2
- U1 pad 11: Net-(U1-P60) -> /Key3
- U1 pad 12: Net-(U1-P61) -> /Key4
- U1 pad 6: Net-(U1-P122/X2/EXCLK) -> /Key1
- U1 pad 7: Net-(U1-P121/X1) -> /Key2
Routing:
- net /Key4: track 0.00 -> 66.6 mm, vias 0 -> 1
- net Net-(U1-P61): track 65.7 -> 0.00 mm, vias 2 -> 0
- net /Key3: track 0.00 -> 62.7 mm, vias 0 -> 2
- net Net-(U1-P60): track 62.4 -> 0.00 mm, vias 2 -> 0
- net /Key1: track 0.00 -> 60.2 mm, vias 0 -> 3
- net Net-(U1-P122/X2/EXCLK): track 57.4 -> 0.00 mm, vias 2 -> 0
- net /Key2: track 0.00 -> 50.5 mm, vias 0 -> 2
- net Net-(U1-P121/X1): track 48.6 -> 0.00 mm, vias 2 -> 0
- net GND: track 109.9 -> 121.2 mm, vias 9 -> 8
- net Net-(P4-Pin_1): track 6.77 -> 0.00 mm
- net Net-(P4-Pin_4): track 6.76 -> 0.00 mm
- net Net-(P4-Pin_2): track 6.76 -> 0.00 mm
- net Net-(P4-Pin_3): track 6.76 -> 0.00 mm
- net +3.3V: track 236.9 -> 242.4 mm, vias 1 -> 2

Commit message: Added a few projects
Routing:
- net +5V: track 73.7 -> 75.4 mm
Changed lines of the file:
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@@
 		(tags "resistor")
 		(property "Reference" "R6"
-			(at 3.05 -0.1 360)
+			(at 3.05 -0.1 0)
 			(layer "F.SilkS")
 			(hide yes)
@@
 		)
 		(property "Value" "10k"
-			(at 6.2 -0.2 360)
+			(at 6.2 -0.2 0)
 			(layer "F.Fab")
 			(hide yes)
@@
 		(tags "resistor")
 		(property "Reference" "R5"
-			(at 0 -1.65 360)
+			(at 0 -1.65 0)
 			(layer "F.SilkS")
 			(hide yes)
@@
 		)
 		(property "Value" "10k"
-			(at 5.95 -0.15 360)
+			(at 5.95 -0.15 0)
 			(layer "F.Fab")
 			(hide yes)
@@
 		(start 131.3042 80.3275)
 		(end 129.3017 78.325)
-		(width 0.25)
+		(width 0.5)
 		(layer "F.Cu")
 		(net 2)
@@
 		(start 128.7384 78.325)
 		(end 129.3017 78.325)
-		(width 0.25)
+		(width 0.5)
 		(layer "F.Cu")
 		(net 2)
@@
 		(start 133.93 80.3275)
 		(end 131.3042 80.3275)
-		(width 0.25)
+		(width 0.5)
 		(layer "F.Cu")
 		(net 2)
@@
 	)
 	(segment
+		(start 128.175 77.025)
+		(end 127.175 76.025)
+		(width 0.5)
+		(layer "B.Cu")
+		(net 2)
+	)
+	(segment
 		(start 142.4733 109.1643)
 		(end 142.4733 114.4084)
@@
 	)
 	(segment
-		(start 118.1278 77.1722)
-		(end 116.55 78.75)
-		(width 0.25)
+		(start 128.175 78.325)
+		(end 128.175 77.025)
+		(width 0.5)
 		(layer "B.Cu")
 		(net 2)
 	)
 	(segment
-		(start 143.6 115.5351)
-		(end 143.6 116.38)
-		(width 0.25)
+		(start 127.175 76.025)
+		(end 119.275 76.025)
+		(width 0.5)
 		(layer "B.Cu")
 		(net 2)
 	)
 	(segment
-		(start 127.0222 77.1722)
-		(end 118.1278 77.1722)
+		(start 143.6 115.5351)
+		(end 143.6 116.38)
 		(width 0.25)
 		(layer "B.Cu")
@@
 	)
 	(segment
-		(start 128.175 78.325)
-		(end 127.0222 77.1722)
-		(width 0.25)
+		(start 119.275 76.025)
+		(end 116.55 78.75)
+		(width 0.5)
 		(layer "B.Cu")
 		(net 2)
@@
 		(start 135.3416 78.0275)
 		(end 133.93 78.0275)
-		(width 0.25)
+		(width 0.5)
 		(layer "F.Cu")
 		(net 4)
@@
 		(start 140.23 78.0275)
 		(end 137.4 78.0275)
-		(width 0.25)
+		(width 0.5)
 		(layer "F.Cu")
 		(net 4)
@@
 		(start 137.4 78.0275)
 		(end 135.3416 78.0275)
-		(width 0.25)
+		(width 0.5)
 		(layer "F.Cu")
 		(net 4)
@@
 		(start 137.4 85.3324)
 		(end 137.4 78.0275)
-		(width 0.25)
+		(width 0.5)
 		(layer "B.Cu")
 		(net 4)
@@
 		(start 134.9 87.8324)
 		(end 137.4 85.3324)
-		(width 0.25)
+		(width 0.5)
 		(layer "B.Cu")
 		(net 4)
